File: schematics/powerfb/powerfb.kicad_sch (KiCad schematic)
At the start: 0 parts

Commit message: backup: pre-reinstall 2026-06-09
Parts:
- added C1, C2, C3, C4, C5, C6, C7, C8, C9: C, symbol Device:C
- added D1, D2, D3: 1N4148WT, Diode_SMD:D_SOD-523, symbol Diode:1N4148WT
- added R1, R2, R3, R4, R5, R6: R, symbol Device:R
- added U1, U2, U3: NE555P, Package_DIP:DIP-8_W7.62mm, symbol Timer:NE555P
Connections:
- new net: C3.1, U2.5 (CONT)
- new net: C9.1, D3.2 (A), U2.3 (OUT)
- new net: R5.2, R6.1, U3.6 (THRES), U3.7 (DISCH)
- new net: C6.1, C9.2, R6.2, U3.2 (TRIG)
- new net: C8.1, D2.2 (A), U3.3 (OUT)
- new net: C1.1, C8.2, R2.2, U1.2 (TRIG)
- new net: C7.1, D1.2 (A), U1.3 (OUT)
- new net: C2.1, U1.5 (CONT)
- new net: R1.2, R2.1, U1.6 (THRES), U1.7 (DISCH)
- new net: C5.1, C7.2, R4.2, U2.2 (TRIG)
- new net: R3.2, R4.1, U2.6 (THRES), U2.7 (DISCH)
- new net: C4.1, U3.5 (CONT)
- new net GND: C1.2, C2.2, C3.2, C4.2, C5.2, C6.2, U1.1 (GND), U2.1 (GND), U3.1 (GND)
- new net VCC: R1.1, R3.1, R5.1, U1.4 (~{RST}), U1.8 (VCC), U2.4 (~{RST}), U2.8 (VCC), U3.4 (~{RST}), U3.8 (VCC)
